File: V1/dc-ac-8ch-v1.kicad_sch (KiCad schematic)
At the start: 8 parts, among them J1 LOAD, J2 NEUTRAL, U1 MOC3031M

Commit message: Circuit under dev
Parts:
- removed J1: LOAD, symbol Connector_Generic:Conn_01x01
- removed J2: NEUTRAL, symbol Connector_Generic:Conn_01x01
- removed U1: MOC3031M, symbol Relay_SolidState:MOC3031M
- added J1: DB142V-5.08-8P, Tales:TerminalBlock_Dibo_DB142V-5.08-8P_1x08_P5.08mm_Vertical, symbol Connector_Generic:Conn_01x08
- added J2: DB142V-5.08-2P, Tales:TerminalBlock_Dibo_DB142V-5.08-2P_1x02_P5.08mm_Vertical, symbol Connector_Generic:Conn_01x02
- added RV1: Varistor, symbol Device:Varistor
- added U2: MOC3063S, Tales:SOP-6_6.6x9.15mm_P2.54mm, symbol Relay_SolidState:MOC3063M
- C1: value C_Small -> 22nF/630V; footprint (none) -> Tales:C_1206_3216Metric; JLCPCB BOM (none) -> 1; LCSC Part # (none) -> C318759; Mfr (none) -> Samsung Electro-Mechanics; Mfr Part # (none) -> CL31B223KHHNNNE; Package (none) -> 1206; Technology (none) -> X7R; Vendor (none) -> JLCPCB; Vendor Part # (none) -> C318759
- D1: value Q_TRIAC_A1A2G -> T435-600B; footprint (none) -> Tales:TO-252-2; JLCPCB BOM (none) -> 1; LCSC Part # (none) -> C145128; Mfr (none) -> STMicroelectronics; Mfr Part # (none) -> T435-600B-TR; Package (none) -> TO-252-2(DPAK); Technology (none) -> Snubberless; Vendor (none) -> JLCPCB; Vendor Part # (none) -> C145128
- R1: value R_US -> 51R/0,25W
- R2: value R_US -> 150R/0,25W
- R3: value R_US -> 390R/0,125W
Connections:
- net NEUTRAL: now reaches C1.2, D1.1 (A1), R3.2
- net NEUTRAL: now also J2.1 (Pin_1), J2.2 (Pin_2), RV1.2
- net LOAD: now reaches D1.2 (A2), R1.1
- net LOAD: now also J1.1 (Pin_1), RV1.1
- net at D1.3 (G), R3.1: now also U2.4
- net at R2.2: now also U2.6
Other:
- note added: "Vpico + 15% mínimo"
- moved on the sheet: C1, D1, R1, R2, R3

Commit message: Under development
Parts:
- added C10, C12, C14, C16, C4, C6, C8: 22nF/630V, Tales:C_1206_3216Metric, symbol Device:C_Small
- added C? (x8): 33nF/50V, Tales:C_0805_2012Metric, symbol Device:C_Small
- added D12, D15, D18, D21, D24, D6, D9: T435-600B, Tales:TO-252-2, symbol Tales:T435-600B
- added D? (x8): GREEN, Tales:LED_0603_1608Metric, symbol Device:LED_Small
- added D? (x8): 9V1/500mW, Tales:D_MiniMELF, symbol Device:D_Zener_Small
- added J1: DB142V-5.08-8P, Tales:TerminalBlock_Dibo_DB142V-5.08-8P_1x08_P5.08mm_Vertical, symbol Connector_Generic:Conn_01x08
- added J2: DB142V-5.08-2P, Tales:TerminalBlock_Dibo_DB142V-5.08-2P_1x02_P5.08mm_Vertical, symbol Connector_Generic:Conn_01x02
- added R10, R15, R20, R25, R30, R35, R40: 51R/250mW, Tales:R_1206_3216Metric, symbol Device:R_US
- added R13, R18, R23, R28, R33, R38, R8: 390R/250mW, Tales:R_1206_3216Metric, symbol Device:R_US
- added R14, R19, R24, R29, R34, R39, R9: 150R/250mW, Tales:R_1206_3216Metric, symbol Device:R_US
- added R? (x8): 1k8/125mW, Tales:R_0805_2012Metric, symbol Device:R_US
- added R? (x8): 5,6k/100mW, Tales:R_0603_1608Metric, symbol Device:R_US
- added RV2, RV3, RV4, RV5, RV6, RV7, RV8: 275VAC, Tales:RV_Disc_D9.50mm_W3.6mm_P5.08mm, symbol Device:Varistor
- added U2, U3, U4, U5, U6, U7, U8: MOC3063S, Tales:SMDIP-6_W9.53mm_Clearance8mm, symbol Relay_SolidState:MOC3063M
- D3: renamed from D1; symbol Device:Q_TRIAC_A1A2G -> Tales:T435-600B
- J3: renamed from J1; Package (none) -> 01x08 P5.08; Technology (none) -> Spring Cage
- J4: renamed from J2; Package (none) -> 01x08 P5.08; Technology (none) -> Spring Cage
- R3: value 390R/0,125W -> 390R/250mW; footprint (none) -> Tales:R_1206_3216Metric; JLCPCB BOM (none) -> 1; LCSC Part # (none) -> C25378; Mfr (none) -> UNI-ROYAL(Uniroyal Elec); Mfr Part # (none) -> 1206W4J0391T5E; Package (none) -> 1206/3216; Technology (none) -> Thick Film; Vendor (none) -> JLCPCB; Vendor Part # (none) -> C25378
- R4: renamed from R2; value 150R/0,25W -> 150R/250mW; footprint (none) -> Tales:R_1206_3216Metric; JLCPCB BOM (none) -> 1; LCSC Part # (none) -> C25353; Mfr (none) -> UNI-ROYAL(Uniroyal Elec); Mfr Part # (none) -> 1206W4J0151T5E; Package (none) -> 1206/3216; Technology (none) -> Thick Film; Vendor (none) -> JLCPCB; Vendor Part # (none) -> C25353
- R5: renamed from R1; value 51R/0,25W -> 51R/250mW; footprint (none) -> Tales:R_1206_3216Metric; JLCPCB BOM (none) -> 1; LCSC Part # (none) -> C18019; Mfr (none) -> UNI-ROYAL(Uniroyal Elec); Mfr Part # (none) -> 1206W4F510JT5E; Package (none) -> 1206/3216; Technology (none) -> Thick Film; Vendor (none) -> JLCPCB; Vendor Part # (none) -> C18019
- RV1: value Varistor -> 275VAC; footprint (none) -> Tales:RV_Disc_D9.50mm_W3.6mm_P5.08mm; JLCPCB BOM (none) -> 1; LCSC Part # (none) -> C2761646; Mfr (none) -> Dersonic; Mfr Part # (none) -> RM07D431KC1IE100; Package (none) -> 12x7.5mm; Technology (none) -> MOV; Vendor (none) -> JLCPCB; Vendor Part # (none) -> C2761646
- U1: renamed from U2; footprint Tales:SOP-6_6.6x9.15mm_P2.54mm -> Tales:SMDIP-6_W9.53mm_Clearance8mm
- renumbered C1 to C2
Connections:
- net NEUTRAL: now also C10.2, C12.2, C14.2, C16.2, C4.2, C6.2, C8.2, D12.1 (A1), D15.1 (A1), D18.1 (A1), D21.1 (A1), D24.1 (A1), D6.1 (A1), D9.1 (A1), R13.2, R18.2, R23.2, R28.2, R33.2, R38.2, R8.2, RV2.2, RV3.2, RV4.2, RV5.2, RV6.2, RV7.2, RV8.2
- net at U1.1: now also D?.2 (A)
- net GND: now reaches U1.2
- net GND: now also C?.2, C?.2, C?.2, C?.2, C?.2, C?.2, C?.2, C?.2, D?.1 (K), D?.1 (K), D?.1 (K), D?.1 (K), D?.1 (K), D?.1 (K), D?.1 (K), D?.1 (K), J2.1 (Pin_1), J2.2 (Pin_2), U2.2, U3.2, U4.2, U5.2, U6.2, U7.2, U8.2
- net at J3.2 (Pin_2): now also D21.2 (A2), R35.1, RV7.1
- net at J3.3 (Pin_3): now also D18.2 (A2), R30.1, RV6.1
- net at J3.4 (Pin_4): now also D15.2 (A2), R25.1, RV5.1
- net at J3.5 (Pin_5): now also D12.2 (A2), R20.1, RV4.1
- net at J3.6 (Pin_6): now also D9.2 (A2), R15.1, RV3.1
- net at J3.7 (Pin_7): now also D6.2 (A2), R10.1, RV2.1
- net at J3.8 (Pin_8): now also D3.2 (A2), R5.1, RV1.1
- removed net LOAD: D3.2 (A2), J3.1 (Pin_1), R5.1, RV1.1
- new net: D?.2 (A), R?.2 (x8)
- new net: C10.1, R24.1, R25.2
- new net: R24.2, U5.6
- new net: D18.3 (G), R28.1, U6.4
- new net: D6.3 (G), R8.1, U2.4
- new net: C?.1, D?.1 (K), R?.1 (x8)
- new net: J1.8 (Pin_8), R?.1, R?.2
- new net: C6.1, R14.1, R15.2
- new net: R14.2, U3.6
- new net: D?.2 (A), U5.1
- new net: D15.3 (G), R23.1, U5.4
- new net: C8.1, R19.1, R20.2
- new net: C16.1, R39.1, R40.2
- new net: D9.3 (G), R13.1, U3.4
- new net: C12.1, R29.1, R30.2
- new net: C14.1, R34.1, R35.2
- new net: R39.2, U8.6
- new net: J1.1 (Pin_1), R?.1, R?.2
- new net: J1.5 (Pin_5), R?.1, R?.2
- new net: J1.4 (Pin_4), R?.1, R?.2
- new net: C4.1, R10.2, R9.1
- new net: R9.2, U2.6
- new net: J1.3 (Pin_3), R?.1, R?.2
- new net: D21.3 (G), R33.1, U7.4
- new net: D?.2 (A), U7.1
- new net: D12.3 (G), R18.1, U4.4
- new net: D?.2 (A), U3.1
- new net: D?.2 (A), U6.1
- new net: D?.2 (A), U8.1
- new net: J1.2 (Pin_2), R?.1, R?.2
- new net: J1.7 (Pin_7), R?.1, R?.2
- new net: D24.2 (A2), J3.1 (Pin_1), R40.1, RV8.1
- new net: D?.2 (A), U2.1
- new net: J1.6 (Pin_6), R?.1, R?.2
- new net: D24.3 (G), R38.1, U8.4
- new net: R29.2, U6.6
- new net: R34.2, U7.6
- new net: R19.2, U4.6
- new net: D?.2 (A), U4.1
Other:
- note removed: "Vpico + 15% mínimo"
- moved on the sheet: C2, D3, J3, J4, R3, R4, R5, RV1, U1

Commit message: Under development
Parts:
- removed J1, J3: DB142V-5.08-8P, Tales:TerminalBlock_Dibo_DB142V-5.08-8P_1x08_P5.08mm_Vertical, symbol Connector_Generic:Conn_01x08
- added J1, J2, J4, J5: DB142V-5.08-4P, symbol Connector_Generic:Conn_01x04
- renumbered J2 to J3, J4 to J6
Connections:
- net at D21.2 (A2), R35.1, RV7.1: now also J5.3 (Pin_3)
- net at D12.2 (A2), R20.1, RV4.1: now also J4.4 (Pin_4)
- net at R?.1, R?.2: now also J2.4 (Pin_4)
- net at D3.2 (A2), R5.1, RV1.1: now also J4.1 (Pin_1)
- net at D9.2 (A2), R15.1, RV3.1: now also J4.3 (Pin_3)
- net at D15.2 (A2), R25.1, RV5.1: now also J5.1 (Pin_1)
- net at R?.1, R?.2: now also J1.1 (Pin_1)
- net at R?.1, R?.2: now also J2.1 (Pin_1)
- net at R?.1, R?.2: now also J1.4 (Pin_4)
- net at R?.1, R?.2: now also J1.3 (Pin_3)
- net at D18.2 (A2), R30.1, RV6.1: now also J5.2 (Pin_2)
- net at D6.2 (A2), R10.1, RV2.1: now also J4.2 (Pin_2)
- net at R?.1, R?.2: now also J1.2 (Pin_2)
- net at R?.1, R?.2: now also J2.3 (Pin_3)
- net at D24.2 (A2), R40.1, RV8.1: now also J5.4 (Pin_4)
- net at R?.1, R?.2: now also J2.2 (Pin_2)

Commit message: Development
Parts:
- J1, J2, J4, J5: footprint (none) -> Tales:TerminalBlock_Dibo_DB142V-5.08-4P_1x04_P5.08mm_Vertical_copy
Connections:
- net at D21.2 (A2), R35.1, RV7.1: now also J5.2 (Pin_2); no longer J5.3 (Pin_3)
- net at D12.2 (A2), R20.1, RV4.1: now also J4.1 (Pin_1); no longer J4.4 (Pin_4)
- net at D3.2 (A2), R5.1, RV1.1: now also J4.4 (Pin_4); no longer J4.1 (Pin_1)
- net at D9.2 (A2), R15.1, RV3.1: now also J4.2 (Pin_2); no longer J4.3 (Pin_3)
- net at D15.2 (A2), R25.1, RV5.1: now also J5.4 (Pin_4); no longer J5.1 (Pin_1)
- net at D18.2 (A2), R30.1, RV6.1: now also J5.3 (Pin_3); no longer J5.2 (Pin_2)
- net at D6.2 (A2), R10.1, RV2.1: now also J4.3 (Pin_3); no longer J4.2 (Pin_2)
- net at D24.2 (A2), R40.1, RV8.1: now also J5.1 (Pin_1); no longer J5.4 (Pin_4)
Changed lines of the file:
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@@
     )
   )
-  (symbol (lib_id "Connector_Generic:Conn_01x04") (at 266.7 69.85 0) (unit 1)
-    (in_bom yes) (on_board yes) (dnp no) (fields_autoplaced)
-    (property "Reference" "J4" (at 266.7 62.23 0)
+  (symbol (lib_id "Connector_Generic:Conn_01x04") (at 266.7 72.39 0) (mirror x) (unit 1)
+    (in_bom yes) (on_board yes) (dnp no)
+    (property "Reference" "J4" (at 266.7 80.01 0)
       (effects (font (size 1.27 1.27)))
     )
-    (property "Value" "DB142V-5.08-4P" (at 266.7 64.77 0)
+    (property "Value" "DB142V-5.08-4P" (at 266.7 77.47 0)
       (effects (font (size 1.27 1.27)))
     )
-    (property "Footprint" "" (at 266.7 69.85 0)
+    (property "Footprint" "Tales:TerminalBlock_Dibo_DB142V-5.08-4P_1x04_P5.08mm_Vertical_copy" (at 266.7 72.39 0)
       (effects (font (size 1.27 1.27)) hide)
     )
-    (property "Datasheet" "~" (at 266.7 69.85 0)
+    (property "Datasheet" "~" (at 266.7 72.39 0)
       (effects (font (size 1.27 1.27)) hide)
     )
@@
     )
   )
-  (symbol (lib_id "Connector_Generic:Conn_01x04") (at 266.7 90.17 0) (unit 1)
-    (in_bom yes) (on_board yes) (dnp no) (fields_autoplaced)
-    (property "Reference" "J5" (at 266.7 82.55 0)
+  (symbol (lib_id "Connector_Generic:Conn_01x04") (at 266.7 92.71 0) (mirror x) (unit 1)
+    (in_bom yes) (on_board yes) (dnp no)
+    (property "Reference" "J5" (at 266.7 100.33 0)
       (effects (font (size 1.27 1.27)))
     )
-    (property "Value" "DB142V-5.08-4P" (at 266.7 85.09 0)
+    (property "Value" "DB142V-5.08-4P" (at 266.7 97.79 0)
       (effects (font (size 1.27 1.27)))
     )
-    (property "Footprint" "" (at 266.7 90.17 0)
+    (property "Footprint" "Tales:TerminalBlock_Dibo_DB142V-5.08-4P_1x04_P5.08mm_Vertical_copy" (at 266.7 92.71 0)
       (effects (font (size 1.27 1.27)) hide)
     )
-    (property "Datasheet" "~" (at 266.7 90.17 0)
+    (property "Datasheet" "~" (at 266.7 92.71 0)
       (effects (font (size 1.27 1.27)) hide)
     )
@@
       (effects (font (size 1.27 1.27)))
     )
-    (property "Footprint" "" (at 25.4 100.33 0)
+    (property "Footprint" "Tales:TerminalBlock_Dibo_DB142V-5.08-4P_1x04_P5.08mm_Vertical_copy" (at 25.4 100.33 0)
       (effects (font (size 1.27 1.27)) hide)
     )
@@
       (effects (font (size 1.27 1.27)))
     )
-    (property "Footprint" "" (at 25.4 80.01 0)
+    (property "Footprint" "Tales:TerminalBlock_Dibo_DB142V-5.08-4P_1x04_P5.08mm_Vertical_copy" (at 25.4 80.01 0)
       (effects (font (size 1.27 1.27)) hide)
     )
